Commit message: Update

File: urdf/my_bot.xacro (robot description, xacro)
@@ -23,5 +23,5 @@
       <origin xyz="0 0 0" rpy=" 0 0 0"/>
       <geometry>
-        <box size=".8 .8 .1"/>
+        <box size=".8 .8 .1" />
       </geometry>
     </collision>

Commit message: Update bot for testing

File: urdf/my_bot.xacro (robot description, xacro)
@@ -23,5 +23,5 @@
       <origin xyz="0 0 0" rpy=" 0 0 0"/>
       <geometry>
-        <box size=".8 .8 .1" />
+        <box size=".8 .8 .1"/>
       </geometry>
     </collision>

Commit message: Update bot for testing

File: urdf/my_bot.xacro (robot description, xacro)
@@ -29,5 +29,5 @@
       <origin xyz="0 0 0" rpy=" 0 0 0"/>
       <geometry>
-        <box size=".8 .9 .5"/>
+        <box size=".8 .8 .1"/>
       </geometry>
     </visual>

Commit message: Update bot for testing

File: urdf/my_bot.xacro (robot description, xacro)
@@ -32,4 +32,5 @@
       </geometry>
     </visual>
+<!--
     <collision name="back_caster_collision">
       <origin xyz="-0.15 0 -0.05" rpy=" 0 0 0"/>
@@ -76,4 +77,43 @@
       </geometry>
     </visual>
+-->
+  </link>
+  <joint name="back_caster_wheel_fixed" type="fixes">
+    <origin xyz="-0.15 0.0 -0.05" rpy="0 0 0"/>
+    <child link="back_caster_wheel"/>
+    <parent link="chassis" />
+  </joint>
+  <link name="back_caster_wheel">
+      <inertial>
+        <mass value="0.1"/>
+        <origin xyz="0.0 0 0" rpy=" 0 0 0"/>
+        <inertia
+            ixx="1e-6" ixy="0" ixz="0"
+            iyy="1e-6" iyz="0"
+            izz="1e-6"
+        />
+      </inertial>
+      <collision>
+        <origin xyz="-0.15 0 -0.05" rpy=" 0 0 0"/>
+        <geometry>
+          <sphere radius="0.05"/>
+        </geometry>
+        <surface>
+          <friction>
+            <ode>
+              <mu>0</mu>
+              <mu2>0</mu2>
+              <slip1>1.0</slip1>
+              <slip2>1.0</slip2>
+            </ode>
+          </friction>
+        </surface>
+      </collision>
+      <visual>
+        <origin xyz="-0.15 0 -0.05" rpy=" 0 0 0"/>
+        <geometry>
+          <sphere radius="0.05"/>
+        </geometry>
+      </visual>
   </link>
   <!-- ====== Wheels ============= -->

Commit message: Update bot for testing

File: urdf/my_bot.xacro (robot description, xacro)
@@ -79,5 +79,5 @@
 -->
   </link>
-  <joint name="back_caster_wheel_fixed" type="fixes">
+  <joint name="back_caster_wheel_fixed" type="fixed">
     <origin xyz="-0.15 0.0 -0.05" rpy="0 0 0"/>
     <child link="back_caster_wheel"/>

Commit message: Update bot for testing

File: urdf/my_bot.xacro (robot description, xacro)
@@ -95,5 +95,5 @@
       </inertial>
       <collision>
-        <origin xyz="-0.15 0 -0.05" rpy=" 0 0 0"/>
+        <origin xyz="0 0 0" rpy="0 0 0"/>
         <geometry>
           <sphere radius="0.05"/>
@@ -111,5 +111,5 @@
       </collision>
       <visual>
-        <origin xyz="-0.15 0 -0.05" rpy=" 0 0 0"/>
+        <origin xyz="0 0 0" rpy="0 0 0"/>
         <geometry>
           <sphere radius="0.05"/>

Commit message: Update bot for testing

File: urdf/my_bot.xacro (robot description, xacro)
@@ -10,5 +10,5 @@
   <!-- ===== Chassis ===== -->
   <link name="chassis">
-    <pose>0 0 0 0 0 0</pose> <!-- 0 0 0.1 0 0 0 -->
+    <pose>0 0 0.1 0 0 0</pose> <!-- 0 0 0.1 0 0 0 -->
     <inertial>
       <mass value="15.0"/>
@@ -117,4 +117,42 @@
       </visual>
   </link>
+  <joint name="dome_fixed" type="fixed">
+    <origin xyz="0 0 0.075" rpy="0 0 0"/>
+    <child link="dome"/>
+    <parent link="chassis" />
+  </joint>
+  <link name="dome">
+      <inertial>
+        <mass value="0.1"/>
+        <origin xyz="0.0 0 0" rpy=" 0 0 0"/>
+        <inertia
+            ixx="1e-6" ixy="0" ixz="0"
+            iyy="1e-6" iyz="0"
+            izz="1e-6"
+        />
+      </inertial>
+      <collision>
+        <origin xyz="0 0 0" rpy="0 0 0"/>
+        <geometry>
+          <box size="0.6 0.6 0.05"/>
+        </geometry>
+        <surface>
+          <friction>
+            <ode>
+              <mu>0</mu>
+              <mu2>0</mu2>
+              <slip1>1.0</slip1>
+              <slip2>1.0</slip2>
+            </ode>
+          </friction>
+        </surface>
+      </collision>
+      <visual>
+        <origin xyz="0 0 0" rpy="0 0 0"/>
+        <geometry>
+          <box size="0.6 0.6 0.05"/>
+        </geometry>
+      </visual>
+  </link>
   <!-- ====== Wheels ============= -->
   <link name="left_wheel">

Commit message: Update bot for testing

File: urdf/my_bot.xacro (robot description, xacro)
@@ -23,5 +23,5 @@
       <origin xyz="0 0 0" rpy=" 0 0 0"/>
       <geometry>
-        <box size=".8 .8 .1"/>
+        <box size=".4 .4 .1"/>
       </geometry>
     </collision>
@@ -29,5 +29,5 @@
       <origin xyz="0 0 0" rpy=" 0 0 0"/>
       <geometry>
-        <box size=".8 .8 .1"/>
+        <box size=".4 .4 .1"/>
       </geometry>
     </visual>
@@ -135,5 +135,5 @@
         <origin xyz="0 0 0" rpy="0 0 0"/>
         <geometry>
-          <box size="0.6 0.6 0.05"/>
+          <box size="0.3 0.3 0.05"/>
         </geometry>
         <surface>
@@ -151,5 +151,5 @@
         <origin xyz="0 0 0" rpy="0 0 0"/>
         <geometry>
-          <box size="0.6 0.6 0.05"/>
+          <box size="0.3 0.3 0.05"/>
         </geometry>
       </visual>

Commit message: Update bot for testing

File: urdf/my_bot.xacro (robot description, xacro)
@@ -117,10 +117,10 @@
       </visual>
   </link>
-  <joint name="dome_fixed" type="fixed">
+  <joint name="dome0_fixed" type="fixed">
     <origin xyz="0 0 0.075" rpy="0 0 0"/>
-    <child link="dome"/>
-    <parent link="chassis" />
-  </joint>
-  <link name="dome">
+    <child link="dome0"/>
+    <parent link="chassis" />
+  </joint>
+  <link name="dome0">
       <inertial>
         <mass value="0.1"/>
@@ -155,5 +155,51 @@
       </visual>
   </link>
+  <joint name="dome1_fixed" type="fixed">
+    <origin xyz="0 0 0.125" rpy="0 0 0"/>
+    <child link="dome1"/>
+    <parent link="dome0" />
+  </joint>
+  <link name="dome1">
+      <inertial>
+        <mass value="0.1"/>
+        <origin xyz="0.0 0 0" rpy=" 0 0 0"/>
+        <inertia
+            ixx="1e-6" ixy="0" ixz="0"
+            iyy="1e-6" iyz="0"
+            izz="1e-6"
+        />
+      </inertial>
+      <collision>
+        <origin xyz="0 0 0" rpy="0 0 0"/>
+        <geometry>
+          <box size="0.2 0.2 0.05"/>
+        </geometry>
+        <surface>
+          <friction>
+            <ode>
+              <mu>0</mu>
+              <mu2>0</mu2>
+              <slip1>1.0</slip1>
+              <slip2>1.0</slip2>
+            </ode>
+          </friction>
+        </surface>
+      </collision>
+      <visual>
+        <origin xyz="0 0 0" rpy="0 0 0"/>
+        <geometry>
+          <box size="0.2 0.2 0.05"/>
+        </geometry>
+      </visual>
+  </link>
   <!-- ====== Wheels ============= -->
+  <joint name="left_wheel_hinge" type="continuous">
+    <origin xyz="0.05 0.13 0" rpy="0 0 0"/>
+    <child link="left_wheel"/>
+    <parent link="chassis" />
+    <axis xyz="0 1 0" rpy="0 0 0" />
+    <limit effort="10000" velocity="1000" />
+    <joint_properties damping="1.0" friction="1.0" />
+  </joint>
   <link name="left_wheel">
     <inertial>
@@ -179,7 +225,7 @@
     </visual>
   </link>
-  <joint name="left_wheel_hinge" type="continuous">
-    <origin xyz="0.05 0.23 0" rpy="0 0 0"/>
-    <child link="left_wheel"/>
+  <joint name="right_wheel_hinge" type="continuous">
+    <origin xyz="0.05 -0.13 0" rpy="0 0 0"/>
+    <child link="right_wheel"/>
     <parent link="chassis" />
     <axis xyz="0 1 0" rpy="0 0 0" />
@@ -210,12 +256,4 @@
     </visual>
   </link>
-  <joint name="right_wheel_hinge" type="continuous">
-    <origin xyz="0.05 -0.23 0" rpy="0 0 0"/>
-    <child link="right_wheel"/>
-    <parent link="chassis" />
-    <axis xyz="0 1 0" rpy="0 0 0" />
-    <limit effort="10000" velocity="1000" />
-    <joint_properties damping="1.0" friction="1.0" />
-  </joint>
   <!-- ====== Camera ============= -->
   <joint name="camera_joint" type="fixed">

Commit message: Update bot for testing

File: urdf/my_bot.xacro (robot description, xacro)
@@ -23,5 +23,5 @@
       <origin xyz="0 0 0" rpy=" 0 0 0"/>
       <geometry>
-        <box size=".4 .4 .1"/>
+        <box size=".4 .4 .05"/>
       </geometry>
     </collision>
@@ -29,5 +29,5 @@
       <origin xyz="0 0 0" rpy=" 0 0 0"/>
       <geometry>
-        <box size=".4 .4 .1"/>
+        <box size=".4 .4 .05"/>
       </geometry>
     </visual>
@@ -156,5 +156,5 @@
   </link>
   <joint name="dome1_fixed" type="fixed">
-    <origin xyz="0 0 0.125" rpy="0 0 0"/>
+    <origin xyz="0 0 0.05" rpy="0 0 0"/>
     <child link="dome1"/>
     <parent link="dome0" />
@@ -193,4 +193,42 @@
       </visual>
   </link>
+  <joint name="dome2_fixed" type="fixed">
+    <origin xyz="0 0 0.05" rpy="0 0 0"/>
+    <child link="dome2"/>
+    <parent link="dome1" />
+  </joint>
+  <link name="dome2">
+      <inertial>
+        <mass value="0.1"/>
+        <origin xyz="0.0 0 0" rpy=" 0 0 0"/>
+        <inertia
+            ixx="1e-6" ixy="0" ixz="0"
+            iyy="1e-6" iyz="0"
+            izz="1e-6"
+        />
+      </inertial>
+      <collision>
+        <origin xyz="0 0 0" rpy="0 0 0"/>
+        <geometry>
+          <box size="0.1 0.1 0.05"/>
+        </geometry>
+        <surface>
+          <friction>
+            <ode>
+              <mu>0</mu>
+              <mu2>0</mu2>
+              <slip1>1.0</slip1>
+              <slip2>1.0</slip2>
+            </ode>
+          </friction>
+        </surface>
+      </collision>
+      <visual>
+        <origin xyz="0 0 0" rpy="0 0 0"/>
+        <geometry>
+          <box size="0.1 0.1 0.05"/>
+        </geometry>
+      </visual>
+  </link>
   <!-- ====== Wheels ============= -->
   <joint name="left_wheel_hinge" type="continuous">

Commit message: Update bot for testing

File: urdf/my_bot.xacro (robot description, xacro)
@@ -32,50 +32,4 @@
       </geometry>
     </visual>
-<!--
-    <collision name="back_caster_collision">
-      <origin xyz="-0.15 0 -0.05" rpy=" 0 0 0"/>
-      <geometry>
-        <sphere radius="0.049"/>
-      </geometry>
-      <surface>
-        <friction>
-          <ode>
-            <mu>0</mu>
-            <mu2>0</mu2>
-            <slip1>1.0</slip1>
-            <slip2>1.0</slip2>
-          </ode>
-        </friction>
-      </surface>
-    </collision>
-    <visual name="back_caster_visual">
-      <origin xyz="-0.15 0 -0.05" rpy=" 0 0 0"/>
-      <geometry>
-        <sphere radius="0.05"/>
-      </geometry>
-    </visual>
-    <collision name="front_caster_collision">
-      <origin xyz="0.15 0 -0.05" rpy=" 0 0 0"/>
-      <geometry>
-        <sphere radius="0.049"/>
-      </geometry>
-      <surface>
-        <friction>
-          <ode>
-            <mu>0</mu>
-            <mu2>0</mu2>
-            <slip1>1.0</slip1>
-            <slip2>1.0</slip2>
-          </ode>
-        </friction>
-      </surface>
-    </collision>
-    <visual name="front_caster_visual">
-      <origin xyz="0.15 0 -0.05" rpy=" 0 0 0"/>
-      <geometry>
-        <sphere radius="0.05"/>
-      </geometry>
-    </visual>
--->
   </link>
   <joint name="back_caster_wheel_fixed" type="fixed">
@@ -118,5 +72,5 @@
   </link>
   <joint name="dome0_fixed" type="fixed">
-    <origin xyz="0 0 0.075" rpy="0 0 0"/>
+    <origin xyz="0 0 0.05" rpy="0 0 0"/>
     <child link="dome0"/>
     <parent link="chassis" />

Commit message: Update bot for testing

File: urdf/my_bot.xacro (robot description, xacro)
@@ -207,5 +207,5 @@
       <origin xyz="0 0 0" rpy="1.5707 0 0"/>
       <geometry>
-        <cylinder radius=".1" length="0.05"/>
+        <cylinder radius=".05" length="0.05"/>
       </geometry>
     </collision>
@@ -213,5 +213,5 @@
       <origin xyz="0 0 0" rpy="1.5707 0 0"/>
       <geometry>
-        <cylinder radius="0.1" length="0.05"/>
+        <cylinder radius="0.05" length="0.05"/>
       </geometry>
     </visual>
@@ -238,5 +238,5 @@
       <origin xyz="0 0 0" rpy="1.5707 0 0"/>
       <geometry>
-        <cylinder radius=".1" length="0.05"/>
+        <cylinder radius=".05" length="0.05"/>
       </geometry>
     </collision>
@@ -244,5 +244,5 @@
       <origin xyz="0 0 0" rpy="1.5707 0 0"/>
       <geometry>
-        <cylinder radius="0.1" length="0.05"/>
+        <cylinder radius="0.05" length="0.05"/>
       </geometry>
     </visual>

Commit message: Update bot for testing

File: urdf/my_bot.xacro (robot description, xacro)
@@ -187,5 +187,5 @@
   <!-- ====== Wheels ============= -->
   <joint name="left_wheel_hinge" type="continuous">
-    <origin xyz="0.05 0.13 0" rpy="0 0 0"/>
+    <origin xyz="0.05 0.13 -0.05" rpy="0 0 0"/>
     <child link="left_wheel"/>
     <parent link="chassis" />
@@ -218,5 +218,5 @@
   </link>
   <joint name="right_wheel_hinge" type="continuous">
-    <origin xyz="0.05 -0.13 0" rpy="0 0 0"/>
+    <origin xyz="0.05 -0.13 -0.05" rpy="0 0 0"/>
     <child link="right_wheel"/>
     <parent link="chassis" />

Commit message: Update bot for testing

File: urdf/my_bot.xacro (robot description, xacro)
@@ -34,5 +34,5 @@
   </link>
   <joint name="back_caster_wheel_fixed" type="fixed">
-    <origin xyz="-0.15 0.0 -0.05" rpy="0 0 0"/>
+    <origin xyz="-0.15 0.0 -0.025" rpy="0 0 0"/>
     <child link="back_caster_wheel"/>
     <parent link="chassis" />
@@ -187,5 +187,5 @@
   <!-- ====== Wheels ============= -->
   <joint name="left_wheel_hinge" type="continuous">
-    <origin xyz="0.05 0.13 -0.05" rpy="0 0 0"/>
+    <origin xyz="0.05 0.13 -0.025" rpy="0 0 0"/>
     <child link="left_wheel"/>
     <parent link="chassis" />
@@ -218,5 +218,5 @@
   </link>
   <joint name="right_wheel_hinge" type="continuous">
-    <origin xyz="0.05 -0.13 -0.05" rpy="0 0 0"/>
+    <origin xyz="0.05 -0.13 -0.025" rpy="0 0 0"/>
     <child link="right_wheel"/>
     <parent link="chassis" />

Commit message: updates

File: urdf/my_bot.xacro (robot description, xacro)
@@ -34,5 +34,5 @@
   </link>
   <joint name="back_caster_wheel_fixed" type="fixed">
-    <origin xyz="-0.15 0.0 -0.025" rpy="0 0 0"/>
+    <origin xyz="-0.1 0.0 -0.025" rpy="0 0 0"/>
     <child link="back_caster_wheel"/>
     <parent link="chassis" />
@@ -147,4 +147,5 @@
       </visual>
   </link>
+<!--
   <joint name="dome2_fixed" type="fixed">
     <origin xyz="0 0 0.05" rpy="0 0 0"/>
@@ -185,7 +186,8 @@
       </visual>
   </link>
+-->
   <!-- ====== Wheels ============= -->
   <joint name="left_wheel_hinge" type="continuous">
-    <origin xyz="0.05 0.13 -0.025" rpy="0 0 0"/>
+    <origin xyz="0.1 0.13 -0.025" rpy="0 0 0"/>
     <child link="left_wheel"/>
     <parent link="chassis" />
@@ -218,5 +220,5 @@
   </link>
   <joint name="right_wheel_hinge" type="continuous">
-    <origin xyz="0.05 -0.13 -0.025" rpy="0 0 0"/>
+    <origin xyz="0.1 -0.13 -0.025" rpy="0 0 0"/>
     <child link="right_wheel"/>
     <parent link="chassis" />
@@ -250,5 +252,5 @@
   <!-- ====== Camera ============= -->
   <joint name="camera_joint" type="fixed">
-    <origin xyz="0.2 0 0" rpy="0 0 0" />
+    <origin xyz="0.15 0 0.04" rpy="0 0 0" />
     <child link="camera" />
     <parent link="chassis" />
@@ -279,5 +281,5 @@
   <!-- ======= Laser Rangefinder ======= -->
   <joint name="hokuyo_joint" type="fixed">
-    <origin xyz=".15 0 .1" />
+    <origin xyz="0 0 .18" /> <!-- .15 0 .3 -->
     <child link="hokuyo" />
     <parent link="chassis" />
