Commit message: updates

File: urdf/my_bot.xacro (robot description, xacro)
@@ -1,5 +1,5 @@
 <?xml version="1.0"?>
 <robot name="my_bot" xmlns:xacro="http://www.ros.org/wiki/xacro">
-  <xacro:include filename="$(find udacity_bot)/urdf/udacity_bot.gazebo" />
+  <xacro:include filename="$(find udacity_bot)/urdf/my_bot.gazebo" />
   <link name="robot_footprint"></link>
   <joint name="robot_footprint_joint" type="fixed">
@@ -23,5 +23,5 @@
       <origin xyz="0 0 0" rpy=" 0 0 0"/>
       <geometry>
-        <box size=".4 .4 .05"/>
+        <box size=".35 .35 .05"/>
       </geometry>
     </collision>
@@ -29,5 +29,5 @@
       <origin xyz="0 0 0" rpy=" 0 0 0"/>
       <geometry>
-        <box size=".4 .4 .05"/>
+        <box size=".35 .35 .05"/>
       </geometry>
     </visual>
@@ -109,8 +109,47 @@
       </visual>
   </link>
+  <!-- head stand -->
+  <joint name="stand_fixed" type="fixed">
+    <origin xyz="0.1 0 0.040" rpy="0 0 0"/>
+    <child link="stand"/>
+    <parent link="dome0" />
+  </joint>
+  <link name="stand">
+      <inertial>
+        <mass value="0.01"/>
+        <origin xyz="0.0 0 0" rpy=" 0 0 0"/>
+        <inertia
+            ixx="1e-7" ixy="0" ixz="0"
+            iyy="1e-7" iyz="0"
+            izz="1e-7"
+        />
+      </inertial>
+      <collision>
+        <origin xyz="0 0 0" rpy="0 0 0"/>
+        <geometry>
+          <cylinder radius=".025" length="0.03"/>
+        </geometry>
+        <surface>
+          <friction>
+            <ode>
+              <mu>0</mu>
+              <mu2>0</mu2>
+              <slip1>1.0</slip1>
+              <slip2>1.0</slip2>
+            </ode>
+          </friction>
+        </surface>
+      </collision>
+      <visual>
+        <origin xyz="0 0 0" rpy="0 0 0"/>
+        <geometry>
+          <cylinder radius=".025" length="0.03"/>
+        </geometry>
+      </visual>
+  </link>
   <joint name="dome1_fixed" type="fixed">
-    <origin xyz="0 0 0.05" rpy="0 0 0"/>
+    <origin xyz="0 0 0.04" rpy="0 0 0"/>
     <child link="dome1"/>
-    <parent link="dome0" />
+    <parent link="stand" />
   </joint>
   <link name="dome1">
@@ -127,64 +166,178 @@
         <origin xyz="0 0 0" rpy="0 0 0"/>
         <geometry>
-          <box size="0.2 0.2 0.05"/>
-        </geometry>
-        <surface>
-          <friction>
-            <ode>
-              <mu>0</mu>
-              <mu2>0</mu2>
-              <slip1>1.0</slip1>
-              <slip2>1.0</slip2>
-            </ode>
-          </friction>
-        </surface>
-      </collision>
-      <visual>
-        <origin xyz="0 0 0" rpy="0 0 0"/>
-        <geometry>
-          <box size="0.2 0.2 0.05"/>
-        </geometry>
-      </visual>
-  </link>
-<!--
-  <joint name="dome2_fixed" type="fixed">
-    <origin xyz="0 0 0.05" rpy="0 0 0"/>
-    <child link="dome2"/>
+          <box size="0.1 0.15 0.05"/>
+        </geometry>
+        <surface>
+          <friction>
+            <ode>
+              <mu>0</mu>
+              <mu2>0</mu2>
+              <slip1>1.0</slip1>
+              <slip2>1.0</slip2>
+            </ode>
+          </friction>
+        </surface>
+      </collision>
+      <visual>
+        <origin xyz="0 0 0" rpy="0 0 0"/>
+        <geometry>
+          <box size="0.1 0.15 0.05"/>
+        </geometry>
+      </visual>
+  </link>
+  <!-- ======= Ears ================= -->
+  <joint name="left_ear_fixed" type="fixed">
+    <origin xyz="0.02 0.075 0" rpy="0 0 0"/>
+    <child link="left_ear"/>
     <parent link="dome1" />
   </joint>
-  <link name="dome2">
-      <inertial>
-        <mass value="0.1"/>
-        <origin xyz="0.0 0 0" rpy=" 0 0 0"/>
-        <inertia
-            ixx="1e-6" ixy="0" ixz="0"
-            iyy="1e-6" iyz="0"
-            izz="1e-6"
-        />
-      </inertial>
-      <collision>
-        <origin xyz="0 0 0" rpy="0 0 0"/>
-        <geometry>
-          <box size="0.1 0.1 0.05"/>
-        </geometry>
-        <surface>
-          <friction>
-            <ode>
-              <mu>0</mu>
-              <mu2>0</mu2>
-              <slip1>1.0</slip1>
-              <slip2>1.0</slip2>
-            </ode>
-          </friction>
-        </surface>
-      </collision>
-      <visual>
-        <origin xyz="0 0 0" rpy="0 0 0"/>
-        <geometry>
-          <box size="0.1 0.1 0.05"/>
-        </geometry>
-      </visual>
-  </link>
--->
+  <link name="left_ear">
+      <inertial>
+        <mass value="0.01"/>
+        <origin xyz="0.0 0 0" rpy=" 0 0 0"/>
+        <inertia
+            ixx="1e-7" ixy="0" ixz="0"
+            iyy="1e-7" iyz="0"
+            izz="1e-7"
+        />
+      </inertial>
+      <collision>
+        <origin xyz="0 0 0" rpy="0 1.5707 0"/>
+        <geometry>
+          <cylinder radius="0.025" length="0.025"/>
+        </geometry>
+        <surface>
+          <friction>
+            <ode>
+              <mu>0</mu>
+              <mu2>0</mu2>
+              <slip1>1.0</slip1>
+              <slip2>1.0</slip2>
+            </ode>
+          </friction>
+        </surface>
+      </collision>
+      <visual>
+        <origin xyz="0 0 0" rpy="0 1.5707 0"/>
+        <geometry>
+          <cylinder radius="0.025" length="0.025"/>
+        </geometry>
+      </visual>
+  </link>
+  <joint name="right_ear_fixed" type="fixed">
+    <origin xyz="0.02 -0.075 0" rpy="0 0 0"/>
+    <child link="right_ear"/>
+    <parent link="dome1" />
+  </joint>
+  <link name="right_ear">
+      <inertial>
+        <mass value="0.01"/>
+        <origin xyz="0.0 0 0" rpy=" 0 0 0"/>
+        <inertia
+            ixx="1e-7" ixy="0" ixz="0"
+            iyy="1e-7" iyz="0"
+            izz="1e-7"
+        />
+      </inertial>
+      <collision>
+        <origin xyz="0 0 0" rpy="0 1.5707 0"/>
+        <geometry>
+          <cylinder radius="0.025" length="0.025"/>
+        </geometry>
+        <surface>
+          <friction>
+            <ode>
+              <mu>0</mu>
+              <mu2>0</mu2>
+              <slip1>1.0</slip1>
+              <slip2>1.0</slip2>
+            </ode>
+          </friction>
+        </surface>
+      </collision>
+      <visual>
+        <origin xyz="0 0 0" rpy="0 1.5707 0"/>
+        <geometry>
+          <cylinder radius="0.025" length="0.025"/>
+        </geometry>
+      </visual>
+  </link>
+  <!-- ======= Eyes =============== -->
+  <joint name="left_eye_fixed" type="fixed">
+    <origin xyz="0.05 0.05 0" rpy="0 0 0"/>
+    <child link="left_eye"/>
+    <parent link="dome1" />
+  </joint>
+  <link name="left_eye">
+      <inertial>
+        <mass value="0.01"/>
+        <origin xyz="0.0 0 0" rpy=" 0 0 0"/>
+        <inertia
+            ixx="1e-7" ixy="0" ixz="0"
+            iyy="1e-7" iyz="0"
+            izz="1e-7"
+        />
+      </inertial>
+      <collision>
+        <origin xyz="0 0 0" rpy="0 1.5707 0"/>
+        <geometry>
+          <cylinder radius="0.012" length="0.01"/>
+        </geometry>
+        <surface>
+          <friction>
+            <ode>
+              <mu>0</mu>
+              <mu2>0</mu2>
+              <slip1>1.0</slip1>
+              <slip2>1.0</slip2>
+            </ode>
+          </friction>
+        </surface>
+      </collision>
+      <visual>
+        <origin xyz="0 0 0" rpy="0 1.5707 0"/>
+        <geometry>
+          <cylinder radius="0.012" length="0.01"/>
+        </geometry>
+      </visual>
+  </link>
+  <joint name="right_eye_fixed" type="fixed">
+    <origin xyz="0.05 -0.05 0" rpy="0 0 0"/>
+    <child link="right_eye"/>
+    <parent link="dome1" />
+  </joint>
+  <link name="right_eye">
+      <inertial>
+        <mass value="0.01"/>
+        <origin xyz="0.0 0 0" rpy=" 0 0 0"/>
+        <inertia
+            ixx="1e-7" ixy="0" ixz="0"
+            iyy="1e-7" iyz="0"
+            izz="1e-7"
+        />
+      </inertial>
+      <collision>
+        <origin xyz="0 0 0" rpy="0 1.5707 0"/>
+        <geometry>
+          <cylinder radius="0.01" length="0.01"/>
+        </geometry>
+        <surface>
+          <friction>
+            <ode>
+              <mu>0</mu>
+              <mu2>0</mu2>
+              <slip1>1.0</slip1>
+              <slip2>1.0</slip2>
+            </ode>
+          </friction>
+        </surface>
+      </collision>
+      <visual>
+        <origin xyz="0 0 0" rpy="0 1.5707 0"/>
+        <geometry>
+          <cylinder radius="0.01" length="0.01"/>
+        </geometry>
+      </visual>
+  </link>
   <!-- ====== Wheels ============= -->
   <joint name="left_wheel_hinge" type="continuous">
@@ -252,5 +405,5 @@
   <!-- ====== Camera ============= -->
   <joint name="camera_joint" type="fixed">
-    <origin xyz="0.15 0 0.04" rpy="0 0 0" />
+    <origin xyz="0.135 0 0.03" rpy="0 0 0" />
     <child link="camera" />
     <parent link="chassis" />
@@ -281,7 +434,7 @@
   <!-- ======= Laser Rangefinder ======= -->
   <joint name="hokuyo_joint" type="fixed">
-    <origin xyz="0 0 .18" /> <!-- .15 0 .3 -->
+    <origin xyz="0 0 .05" /> <!-- .15 0 .3 -->
     <child link="hokuyo" />
-    <parent link="chassis" />
+    <parent link="dome1" />
   </joint>
   <link name="hokuyo">
