Commit message: looks like it works

File: urdf/udacity_bot.xacro (robot description, xacro)
@@ -102,5 +102,5 @@
   </link>
   <joint name="left_wheel_hinge" type="continuous">
-    <origin xyz="0.05 0.13 0" rpy="0 0 0"/>
+    <origin xyz="0.0 0.13 0" rpy="0 0 0"/>
     <child link="left_wheel"/>
     <parent link="chassis" />
@@ -133,5 +133,5 @@
   </link>
   <joint name="right_wheel_hinge" type="continuous">
-    <origin xyz="0.05 -0.13 0" rpy="0 0 0"/>
+    <origin xyz="0.0 -0.13 0" rpy="0 0 0"/>
     <child link="right_wheel"/>
     <parent link="chassis" />
@@ -171,5 +171,5 @@
   <!-- ======= Laser Rangefinder ======= -->
   <joint name="hokuyo_joint" type="fixed">
-    <origin xyz=".15 0 .1" />
+    <origin xyz=".15 0 .2" />
     <child link="hokuyo" />
     <parent link="chassis" />
